File: PCB/keaboard_rev2/keaboard_rev2.kicad_pcb (KiCad board)
At the start: 2 copper layers, 141.9 x 93.7 mm, 88 parts, among them J1 AudioJack4, P1 OLED, P2 LED, SW1 SW_Push, SW10 SW_Push, SW11 SW_Push, SW12 SW_Push, SW13 SW_Push, SW14 SW_Push, SW15 SW_Push, SW16 SW_Push, SW17 SW_Push, SW18 SW_Push, SW19 SW_Push, SW2 SW_Push, SW20 SW_Push, SW21 SW_Push, SW22 SW_Push, SW23 SW_Push, SW24 SW_Push, SW25 SW_Push, SW3 SW_Push, SW4 SW_Push, SW5 SW_Push, SW6 SW_Push, SW7 SW_Push, SW8 SW_Push, SW9 SW_Push, U1 ProMicro

Commit message: WIP
Parts:
- removed the LED19 at (196.5, 100.7)
- added D13: D, Keebio-Parts:Diode-dual, F.Cu at (62.1, 92.2)
- added D14: D, Keebio-Parts:Diode-dual, F.Cu at (81.2, 89.7)
- added D15: D, Keebio-Parts:Diode-dual, F.Cu at (100.2, 87.1)
- added D16: D, Keebio-Parts:Diode-dual, F.Cu at (119.3, 84.6)
- added D17: D, Keebio-Parts:Diode-dual, F.Cu at (138.3, 87.1)
- added D18: D, Keebio-Parts:Diode-dual, F.Cu at (157.4, 89.7)
- added LED25: SK6812MINI-E, parts:SK6812MINI-E_reversible, F.Cu at (198.0, 124.2)
- added LED26: SK6812MINI-E, parts:SK6812MINI-E_reversible, F.Cu at (54.5, 128.6)
- added LED27: SK6812MINI-E, parts:SK6812MINI-E_reversible, F.Cu at (73.5, 126.1)
- added LED28: SK6812MINI-E, parts:SK6812MINI-E_reversible, F.Cu at (92.6, 123.5)
- added LED29: SK6812MINI-E, parts:SK6812MINI-E_reversible, F.Cu at (111.6, 121.0)
- added LED30: SK6812MINI-E, parts:SK6812MINI-E_reversible, F.Cu at (138.8, 125.8)
- added LED31: SK6812MINI-E, parts:SK6812MINI-E_reversible, F.Cu at (198.0, 143.2)
- added SW13: SW_Push, keyswitches:Kailh_socket_PG1350_reversible, F.Cu at (54.5, 95.3)
- added SW14: SW_Push, keyswitches:Kailh_socket_PG1350_reversible, F.Cu at (73.5, 92.7)
- added SW15: SW_Push, keyswitches:Kailh_socket_PG1350_reversible, F.Cu at (92.6, 90.2)
- added SW16: SW_Push, keyswitches:Kailh_socket_PG1350_reversible, F.Cu at (111.6, 87.6)
- added SW17: SW_Push, keyswitches:Kailh_socket_PG1350_reversible, F.Cu at (130.7, 90.2)
- added SW18: SW_Push, keyswitches:Kailh_socket_PG1350_reversible, F.Cu at (149.7, 92.7)
- moved LED24 48.5 mm to (149.7, 107.0)
- moved D31 23.5 mm to (205.6, 144.9)
- moved SW31 23.5 mm to (198.0, 148.0)
- moved D25 23.5 mm to (205.6, 125.9)
- moved SW25 23.5 mm to (198.0, 128.9)
- moved D19 19.1 mm to (62.1, 111.3)
- moved D21 19.1 mm to (100.2, 106.2)
- moved D23 19.1 mm to (138.3, 106.2)
- moved SW19 19.1 mm to (54.5, 114.3)
- moved SW28 19.1 mm to (92.6, 128.3)
- moved SW30 19.1 mm to (138.8, 130.5)
- moved D20 19.0 mm to (81.2, 108.7)
- moved D22 19.0 mm to (119.3, 103.6)
- moved D24 19.0 mm to (157.4, 108.7)
- moved D27 19.0 mm to (81.2, 127.8)
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- renumbered D13 to D19, D14 to D20, D15 to D21, D16 to D22, D17 to D23, D18 to D24, D19 to D25, D20 to D26, D21 to D27, D22 to D28, D23 to D29, D24 to D30, D25 to D31, LED20 to LED19, LED21 to LED20, LED22 to LED21, LED23 to LED22, LED24 to LED23, LED25 to LED24, SW13 to SW19, SW14 to SW20, SW15 to SW21, SW16 to SW22, SW17 to SW23, SW18 to SW24, SW19 to SW25, SW20 to SW26, SW21 to SW27, SW22 to SW28, SW23 to SW29, SW24 to SW30, SW25 to SW31
Connections:
- D19 pad 1: Row2 -> Row3
- D20 pad 1: Row2 -> Row3
- D21 pad 1: Row2 -> Row3
- D22 pad 1: Row2 -> Row3
- D23 pad 1: Row2 -> Row3
- D24 pad 1: Row2 -> Row3
- D25 pad 1: Row2 -> Row3
- D26 pad 1: Row3 -> Row4
- D27 pad 1: Row3 -> Row4
- D28 pad 1: Row3 -> Row4
- D29 pad 1: Row3 -> Row4
- D30 pad 1: Row3 -> Row4
- D31 pad 1: Row3 -> Row4
- LED18 pad 4: Net-(LED18-Pad4) -> Net-(LED12-Pad2)
- U1 pad 11: Net-(U1-Pad11) -> Row4
Routing:
- net Row2: track 106.3 -> 0.00 mm
- net Row1: track 106.3 -> 0.00 mm
- net Row0: track 105.1 -> 0.00 mm
- net Col0: track 100.7 -> 0.00 mm, vias 4 -> 0
- net Col3: track 100.7 -> 0.00 mm, vias 4 -> 0
- net Col2: track 100.7 -> 0.00 mm, vias 4 -> 0
- net Col1: track 100.7 -> 0.00 mm, vias 4 -> 0
- net Col4: track 78.3 -> 0.00 mm, vias 4 -> 0
- net Col5: track 70.2 -> 0.00 mm, vias 3 -> 0
- net Row3: track 66.1 -> 0.00 mm
- net Net-(D25-Pad2): track 21.8 -> 0.00 mm
- net Net-(D12-Pad2): track 21.8 -> 0.00 mm
- net Net-(D8-Pad2): track 21.8 -> 0.00 mm
- net Net-(D26-Pad2): track 21.8 -> 0.00 mm
- net Net-(D6-Pad2): track 21.8 -> 0.00 mm
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Other:
- board size 141.9 x 93.7 mm -> 141.9 x 112.8 mm
